Commit message: reworked controls to get the speed I wanted. reworking rewards. working in the debug visuals. need to actually debug reward

File: onshape_robot/foosball_robot/foosball_robot.urdf (robot description, URDF)
Before this commit: robot foosball_robot, 3 links, 2 joints
Links:
- added link player_2, mass 0.154321; collision mesh filename=package://assets/player.stl; visual mesh filename=package://assets/player.stl
- added link rod_2, mass 0.688975; collision mesh filename=package://assets/rod.stl; visual mesh filename=package://assets/rod.stl
- link main_body: geometry collision mesh filename=package://assets/main_body.stl; visual mesh filename=package://assets/main_body.stl
Joints:
- added joint opponent_kicker: type revolute, parent rod_2, child player_2, origin xyz=8.32667e-17 6.93889e-17 -0.45 rpy=3.14159 -2.34268e-31 -2.55449, axis 0 0 1, limit lower=-3.141592653589793 upper=3.141592653589793 effort=10 velocity=10
- added joint opponent_slider: type prismatic, parent main_body, child rod_2, origin xyz=0.172 -0.453029 0.12 rpy=1.5708 -3.99333e-20 2.92256e-16, axis 0 0 1, limit lower=-0.157029 upper=0.150971 effort=10 velocity=10
- joint kicker: origin xyz=0 0 -0.45 rpy=3.14159 2.13707e-27 -0.785315 -> xyz=-2.77556e-17 5.55112e-17 -0.45 rpy=3.14159 2.13707e-27 -0.785315
- joint slider: limit lower=-0.165237 upper=0.142763 effort=10 velocity=10 -> lower=0 upper=0.308 effort=10 velocity=10; origin xyz=-0.172 -0.461237 0.11 rpy=1.5708 -0 -1.81068e-29 -> xyz=-0.172 -0.296 0.12 rpy=1.5708 -0 -1.81068e-29

Commit message: "selfplay" training working. just two goalies blocking balls, while observing opponent.

File: onshape_robot/foosball_robot/foosball_robot.urdf (robot description, URDF)
Before this commit: robot foosball_robot, 5 links, 4 joints
Joints:
- joint kicker: limit lower=-3.141592653589793 upper=3.141592653589793 effort=10 velocity=10 -> effort=100 velocity=170; origin xyz=-2.77556e-17 5.55112e-17 -0.45 rpy=3.14159 2.13707e-27 -0.785315 -> xyz=-2.77556e-17 6.93889e-17 -0.45 rpy=3.14159 0 0; type revolute -> continuous
- joint opponent_kicker: limit lower=-3.141592653589793 upper=3.141592653589793 effort=10 velocity=10 -> effort=100 velocity=170; origin xyz=8.32667e-17 6.93889e-17 -0.45 rpy=3.14159 -2.34268e-31 -2.55449 -> xyz=-2.77556e-17 1.19349e-15 -0.45 rpy=3.14159 0 0; type revolute -> continuous
- joint opponent_slider: limit lower=-0.157029 upper=0.150971 effort=10 velocity=10 -> lower=-0.154 upper=0.154 effort=100 velocity=15; origin xyz=0.172 -0.453029 0.12 rpy=1.5708 -3.99333e-20 2.92256e-16 -> xyz=0.172 -0.45 0.12 rpy=1.5708 -2.396e-19 4.73315e-30
- joint slider: limit lower=0 upper=0.308 effort=10 velocity=10 -> lower=-0.154 upper=0.154 effort=100 velocity=15; origin xyz=-0.172 -0.296 0.12 rpy=1.5708 -0 -1.81068e-29 -> xyz=-0.172 -0.45 0.12 rpy=1.5708 -1.60236e-18 -2.18272e-28
