Commit message: updated urdf and sim core to be continuous paddle joint

File: onshape_robot/shootout_robot/shootout_robot.urdf (robot description, URDF)
Before this commit: robot shootout_robot, 5 links, 4 joints
Joints:
- joint opponent_paddle: limit lower=-3.141592653589793 upper=3.141592653589793 effort=10 velocity=10 -> effort=10 velocity=10; type revolute -> continuous
- joint paddle: limit lower=-3.141592653589793 upper=3.141592653589793 effort=10 velocity=10 -> effort=10 velocity=10; type revolute -> continuous
